File: projects/przystawka/przystawka/schemat.sch (EAGLE design)
At the start: 51 parts, among them IC1 ESP32-WROOM-32E_M113EH2800PH3Q

Commit message: Editing project teensy4.1 cnc board
Parts:
- removed C3, C4, C5, C6, C7, C8, C9: 100nf, rcl:C-EUC0805
- removed JPP, JPP1, JPP2, JPP3: (no value), pinhead:PINHD-1X2
- removed OK2, OK3, OK4, OK5, OK6, OK7, OK8: 6N137, optocoupler:6N137
- removed R10, R11, R12, R13, R14, R15, R16, R3, R4, R5, R6, R7, R8, R9: 10K, rcl:R-EU_R0805
- added 1, 2, 3, 4, 5, ENDSTOP_JP, VCC5.0_SOCKET3, VCC5.0_SOCKET4: (no value), pinhead:PINHD-1X2
- added 6N137_ME, 6N137_PY, 6N137_PZ, 6N137_SA, 6N137_SPINDLE_OUT, 6N137_XCW, 6N137_YCW, 6N137_ZCW: 6N137, optocoupler:6N137
- added C3Y, C4Z, C5ME, C6XCW, C7YCW, C8SA, C8ZCW, C9S: 100nf, rcl:C-EUC0805
- added FUSE, FUSE1, FUSE2: 200mA, rcl:R-EU_R2512
- added R10XCW, R11YCW, R12YCW, R13SA, R13ZCW, R14SA, R14ZCW, R15S, R16S, R3Y, R4Y, R5Z, R6Z, R7ME, R8ME, R9XCW: 10K, rcl:R-EU_R0805
- renumbered C2 to C2X, JP3 to JP_POWER_IN, JP4 to JP_RX0_TX0_ESP_OUT, JP5 to JP_3V3_EN_ESP_OUT, JP6 to JP_5V_TEENSY_INPUT_ENABLE, OK1 to 6N137_PX, R1 to R1X, R2 to R2X
Connections:
- new net N$13: FUSE.1, JP_5V_TEENSY_INPUT_ENABLE.1
- new net N$14: C1.2, FUSE1.2, FUSE2.2, IC1.3V3, JP_3V3_EN_ESP_OUT.1
- new net N$15: 6N137_SA.VE, R13SA.1
- new net SA: 5.1, 6N137_SA.VO, R14SA.1
- net ENABLE_MOTORS: now also 6N137_ME.A; no longer OK4.A
- net END_STOP_X: now also ENDSTOP_JP.2
- net END_STOP_Y: now also ENDSTOP_JP.1
- net GND: now also 4.2, 6N137_ME.C, 6N137_ME.GND, 6N137_PY.C, 6N137_PY.GND, 6N137_PZ.C, 6N137_PZ.GND, 6N137_SA.C, 6N137_SA.GND, 6N137_SPINDLE_OUT.C, 6N137_SPINDLE_OUT.GND, 6N137_XCW.C, 6N137_XCW.GND, 6N137_YCW.C, 6N137_YCW.GND, 6N137_ZCW.C, 6N137_ZCW.GND, C3Y.2, C4Z.2, C5ME.2, C6XCW.2, C7YCW.2, C8SA.2, C8ZCW.2, C9S.2; no longer C3.2, C4.2, C5.2, C6.2, C7.2, C8.2, C9.2, OK2.C, OK2.GND, OK3.C, OK3.GND, OK4.C, OK4.GND, OK5.C, OK5.GND, OK6.C, OK6.GND, OK7.C, OK7.GND, OK8.C, OK8.GND
- net MOTOR_OUT: now also 5.2, 6N137_ME.VO, R8ME.1; no longer JPP1.2, OK4.VO, R8.1
- net N$10: now also 6N137_XCW.VE, R9XCW.1; no longer OK5.VE, R9.1
- net N$11: now also 6N137_YCW.VE, R11YCW.1; no longer OK6.VE, R11.1
- net N$12: now also 6N137_ZCW.VE, R13ZCW.1; no longer OK7.VE, R13.1
- net N$6: now also 6N137_PY.VE, R3Y.1; no longer OK2.VE, R3.1
- net N$7: now also 6N137_PZ.VE, R5Z.1; no longer OK3.VE, R5.1
- net N$8: now also 6N137_ME.VE, R7ME.1; no longer OK4.VE, R7.1
- net N$9: now also 6N137_SPINDLE_OUT.VE, R15S.1; no longer OK8.VE, R15.1
- net PX_OUT: now also 1.1; no longer JPP.1
- net PY: now also 6N137_PY.A; no longer OK2.A
- net PY_OUT: now also 2.1, 6N137_PY.VO, R4Y.1; no longer JPP.2, OK2.VO, R4.1
- net PZ: now also 6N137_PZ.A; no longer OK3.A
- net PZ_OUT: now also 3.1, 6N137_PZ.VO, R6Z.1; no longer JPP1.1, OK3.VO, R6.1
- net SPINDLE_ANALOG: now also 6N137_SA.A
- net SPINDLE_ENABLE: now also 6N137_SPINDLE_OUT.A; no longer OK8.A
- net SPINDLE_OUT: now also 4.1, 6N137_SPINDLE_OUT.VO, R16S.1; no longer JPP3.2, OK8.VO, R16.1
- net VCC3.3: now also FUSE1.1, FUSE2.1; no longer C1.2, IC1.3V3, JP_3V3_EN_ESP_OUT.1
- net VCC5.0: now also 6N137_ME.VCC, 6N137_PY.VCC, 6N137_PZ.VCC, 6N137_SA.VCC, 6N137_SPINDLE_OUT.VCC, 6N137_XCW.VCC, 6N137_YCW.VCC, 6N137_ZCW.VCC, C3Y.1, C4Z.1, C5ME.1, C6XCW.1, C7YCW.1, C8SA.1, C8ZCW.1, C9S.1, FUSE.2, R10XCW.2, R11YCW.2, R12YCW.2, R13SA.2, R13ZCW.2, R14SA.2, R14ZCW.2, R15S.2, R16S.2, R3Y.2, R4Y.2, R5Z.2, R6Z.2, R7ME.2, R8ME.2, R9XCW.2, VCC5.0_SOCKET3.1, VCC5.0_SOCKET3.2, VCC5.0_SOCKET4.1, VCC5.0_SOCKET4.2; no longer C3.1, C4.1, C5.1, C6.1, C7.1, C8.1, C9.1, JP_5V_TEENSY_INPUT_ENABLE.1, OK2.VCC, OK3.VCC, OK4.VCC, OK5.VCC, OK6.VCC, OK7.VCC, OK8.VCC, R10.2, R11.2, R12.2, R13.2, R14.2, R15.2, R16.2, R3.2, R4.2, R5.2, R6.2, R7.2, R8.2, R9.2
- net XCW: now also 6N137_XCW.A; no longer OK5.A
- net XCW_OUT: now also 1.2, 6N137_XCW.VO, R10XCW.1; no longer JPP2.1, OK5.VO, R10.1
- net YCW: now also 6N137_YCW.A; no longer OK6.A
- net YCW_OUT: now also 2.2, 6N137_YCW.VO, R12YCW.1; no longer JPP2.2, OK6.VO, R12.1
- net ZCW: now also 6N137_ZCW.A; no longer OK7.A
- net ZCW_OUT: now also 3.2, 6N137_ZCW.VO, R14ZCW.1; no longer JPP3.1, OK7.VO, R14.1
