File: projects/przystawka/przystawka/schemat.brd (EAGLE design)
At the start: 133.3 x 105.1 mm, 62 parts, among them IC1 ESP32-WROOM-32E_M113EH2800PH3Q

Commit message: Update schemat and board
Parts:
- moved C9S 3.81 mm to (71.1, 8.89)
- moved R15S 3.81 mm to (71.1, 11.4)
- moved R16S 3.81 mm to (68.6, 6.35)
- moved 6N137_SPINDLE_OUT 3.81 mm to (80.0, 12.7)
Routing:
- net TX2: track 171.1 -> 149.4 mm
- net SPINDLE_ENABLE: track 88.0 -> 75.8 mm
- net RX2: track 153.0 -> 141.6 mm
- net SA: track 31.3 -> 27.1 mm
- net END_STOP_X: track 31.5 -> 28.4 mm
- net XCW_OUT: track 28.3 -> 26.0 mm
- net END_STOP_Y: track 27.2 -> 25.2 mm
- net YCW_OUT: track 28.0 -> 26.0 mm
- net ZCW_OUT: track 27.5 -> 25.5 mm
- net MOTOR_OUT: track 25.4 -> 23.5 mm
- net SPINDLE_OUT: track 59.5 -> 61.1 mm
- net PY_OUT: track 25.6 -> 24.5 mm
- net PZ_OUT: track 25.9 -> 25.0 mm
- net VCC5.0: track 436.4 -> 437.1 mm
- net N$9: track 11.0 -> 10.3 mm
- added copper zone on layer 16, net GND
Other:
- board size 133.3 x 105.1 mm -> 130.8 x 98.7 mm
